Commit message: updated robot desc and movement

File: description/robot_core_lr.xacro (robot description, xacro)
@@ -7,8 +7,9 @@
 	<xacro:property name="mu2" value="550"/>
 	<xacro:property name="velocity" value="1"/>
-	<xacro:property name="effort" value="30"/>
+	<xacro:property name="effort" value="10"/>
 	<xacro:property name="base_mass" value="10"/>
 	<xacro:property name="leg_mass" value="5"/>
-	<xacro:property name="fdir" value="0 1 0"/>
+	<xacro:property name="leg_mass3" value="5"/>
+	<xacro:property name="fdir" value="1 0 0"/>
 	<link name="base_link">
 	</link>
@@ -40,4 +41,7 @@
 		<mu1 value="${mu1}"/>
 		<mu2 value="${mu2}"/>
+		<fdir1 value="${fdir}"/>
+		<maxVel>1.0</maxVel>
+    	<minDepth>0.01</minDepth>
 	</gazebo>
 	<!-- LEFT_LEG1_AX1 -->
@@ -64,5 +68,5 @@
 		</collision>
 		<xacro:inertial_box mass="${leg_mass}" x="0.04" y="0.04" z="0.1">
-			<origin xyz="0 0 0" rpy="0 0 0"/>
+			<origin xyz="0 0 -0.03" rpy="0 0 0"/>
 		</xacro:inertial_box>
 	</link>
@@ -71,4 +75,7 @@
 		<mu1 value="${mu1}"/>
 		<mu2 value="${mu2}"/>
+		<fdir1 value="${fdir}"/>
+		<maxVel>1.0</maxVel>
+    	<minDepth>0.01</minDepth>
 	</gazebo>
 	<!-- LEFT_LEG1_AX2 -->
@@ -95,5 +102,5 @@
 		</collision>
 		<xacro:inertial_box mass="${leg_mass}" x="0.04" y="0.04" z="0.4">
-			<origin xyz="0 0 0" rpy="0 0 0"/>
+			<origin xyz="0 0 0.18" rpy="0 0 0"/>
 		</xacro:inertial_box>
 	</link>
@@ -102,4 +109,7 @@
 		<mu1 value="${mu1}"/>
 		<mu2 value="${mu2}"/>
+		<fdir1 value="${fdir}"/>
+		<maxVel>1.0</maxVel>
+    	<minDepth>0.01</minDepth>
 	</gazebo>
 	<!-- LEFT_LEG1_AX3 -->
@@ -125,19 +135,6 @@
 			</geometry>
 		</collision>
-		<!-- added pads -->
-		<visual>
-			<origin xyz="0 -0.04 0.38"/>
-			<geometry>
-				<sphere radius="0.04"/>
-			</geometry>
-		</visual>
-		<collision>
-			<origin xyz="0 -0.04 0.38"/>
-			<geometry>
-				<sphere radius="0.04"/>
-			</geometry>
-		</collision>
-		<xacro:inertial_box mass="${leg_mass}" x="0.04" y="0.04" z="0.4">
-			<origin xyz="0 0 0" rpy="0 0 0"/>
+		<xacro:inertial_box mass="${leg_mass3}" x="0.04" y="0.04" z="0.4">
+			<origin xyz="0 -0.04 0.18" rpy="0 0 0"/>
 		</xacro:inertial_box>
 	</link>
@@ -147,4 +144,8 @@
 		<mu2 value="${mu2}"/>
 		<fdir1 value="${fdir}"/>
+		<maxVel>1.0</maxVel>
+    	<minDepth>0.01</minDepth>
+		<kp>1000000.0</kp>
+		<kd>100.0</kd>
 	</gazebo>
 	<!-- LEFT_LEG2_AX1 -->
@@ -171,5 +172,5 @@
 		</collision>
 		<xacro:inertial_box mass="${leg_mass}" x="0.04" y="0.04" z="0.1">
-			<origin xyz="0 0 0" rpy="0 0 0"/>
+			<origin xyz="0 0 -0.03" rpy="0 0 0"/>
 		</xacro:inertial_box>
 	</link>
@@ -178,4 +179,7 @@
 		<mu1 value="${mu1}"/>
 		<mu2 value="${mu2}"/>
+		<fdir1 value="${fdir}"/>
+		<maxVel>1.0</maxVel>
+    	<minDepth>0.01</minDepth>
 	</gazebo>
 	<!-- LEFT_LEG2_AX2 -->
@@ -202,5 +206,5 @@
 		</collision>
 		<xacro:inertial_box mass="${leg_mass}" x="0.04" y="0.04" z="0.4">
-			<origin xyz="0 0 0" rpy="0 0 0"/>
+			<origin xyz="0 0 0.18" rpy="0 0 0"/>
 		</xacro:inertial_box>
 	</link>
@@ -209,4 +213,7 @@
 		<mu1 value="${mu1}"/>
 		<mu2 value="${mu2}"/>
+		<fdir1 value="${fdir}"/>
+		<maxVel>1.0</maxVel>
+    	<minDepth>0.01</minDepth>
 	</gazebo>
 	<!-- LEFT_LEG2_AX3 -->
@@ -232,5 +239,5 @@
 			</geometry>
 		</collision>
-		<!-- added pads -->
+		<!-- added pads
 		<visual>
 			<origin xyz="0 -0.04 0.38"/>
@@ -245,6 +252,7 @@
 			</geometry>
 		</collision>
-		<xacro:inertial_box mass="${leg_mass}" x="0.04" y="0.04" z="0.4">
-			<origin xyz="0 0 0" rpy="0 0 0"/>
+		-->
+		<xacro:inertial_box mass="${leg_mass3}" x="0.04" y="0.04" z="0.4">
+			<origin xyz="0 -0.04 0.18" rpy="0 0 0"/>
 		</xacro:inertial_box>
 	</link>
@@ -254,4 +262,8 @@
 		<mu2 value="${mu2}"/>
 		<fdir1 value="${fdir}"/>
+		<maxVel>1.0</maxVel>
+    	<minDepth>0.01</minDepth>
+		<kp>1000000.0</kp>
+		<kd>100.0</kd>
 	</gazebo>
 	<!-- RIGHT_LEG1_AX1 -->
@@ -278,5 +290,5 @@
 		</collision>
 		<xacro:inertial_box mass="${leg_mass}" x="0.04" y="0.04" z="0.1">
-			<origin xyz="0 0 0" rpy="0 0 0"/>
+			<origin xyz="0 0 -0.03" rpy="0 0 0"/>
 		</xacro:inertial_box>
 	</link>
@@ -285,4 +297,7 @@
 		<mu1 value="${mu1}"/>
 		<mu2 value="${mu2}"/>
+		<fdir1 value="${fdir}"/>
+		<maxVel>1.0</maxVel>
+    	<minDepth>0.01</minDepth>
 	</gazebo>
 	<!-- RIGHT_LEG1_AX2 -->
@@ -309,5 +324,5 @@
 		</collision>
 		<xacro:inertial_box mass="${leg_mass}" x="0.04" y="0.04" z="0.4">
-			<origin xyz="0 0 0" rpy="0 0 0"/>
+			<origin xyz="0 0 0.18" rpy="0 0 0"/>
 		</xacro:inertial_box>
 	</link>
@@ -316,4 +331,7 @@
 		<mu1 value="${mu1}"/>
 		<mu2 value="${mu2}"/>
+		<fdir1 value="${fdir}"/>
+		<maxVel>1.0</maxVel>
+    	<minDepth>0.01</minDepth>
 	</gazebo>
 	<!-- RIGHT_LEG1_AX3 -->
@@ -339,5 +357,5 @@
 			</geometry>
 		</collision>
-		<!-- added pads -->
+		<!-- added pads
 		<visual>
 			<origin xyz="0 -0.04 0.38"/>
@@ -352,6 +370,7 @@
 			</geometry>
 		</collision>
-		<xacro:inertial_box mass="${leg_mass}" x="0.04" y="0.04" z="0.4">
-			<origin xyz="0 0 0" rpy="0 0 0"/>
+		-->
+		<xacro:inertial_box mass="${leg_mass3}" x="0.04" y="0.04" z="0.4">
+			<origin xyz="0 -0.04 0.18" rpy="0 0 0"/>
 		</xacro:inertial_box>
 	</link>
@@ -361,4 +380,8 @@
 		<mu2 value="${mu2}"/>
 		<fdir1 value="${fdir}"/>
+		<maxVel>1.0</maxVel>
+    	<minDepth>0.01</minDepth>
+		<kp>1000000.0</kp>
+		<kd>100.0</kd>
 	</gazebo>
 	<!-- RIGHT_LEG2_AX1 -->
@@ -385,5 +408,5 @@
 		</collision>
 		<xacro:inertial_box mass="${leg_mass}" x="0.04" y="0.04" z="0.1">
-			<origin xyz="0 0 0" rpy="0 0 0"/>
+			<origin xyz="0 0 -0.03" rpy="0 0 0"/>
 		</xacro:inertial_box>
 	</link>
@@ -392,4 +415,7 @@
 		<mu1 value="${mu1}"/>
 		<mu2 value="${mu2}"/>
+		<fdir1 value="${fdir}"/>
+		<maxVel>1.0</maxVel>
+    	<minDepth>0.01</minDepth>
 	</gazebo>
 	<!-- RIGHT_LEG2_AX2 -->
@@ -416,5 +442,5 @@
 		</collision>
 		<xacro:inertial_box mass="${leg_mass}" x="0.04" y="0.04" z="0.4">
-			<origin xyz="0 0 0" rpy="0 0 0"/>
+			<origin xyz="0 0 0.18" rpy="0 0 0"/>
 		</xacro:inertial_box>
 	</link>
@@ -423,4 +449,7 @@
 		<mu1 value="${mu1}"/>
 		<mu2 value="${mu2}"/>
+		<fdir1 value="${fdir}"/>
+		<maxVel>1.0</maxVel>
+    	<minDepth>0.01</minDepth>
 	</gazebo>
 	<!-- RIGHT_LEG2_AX3 -->
@@ -446,5 +475,5 @@
 			</geometry>
 		</collision>
-		<!-- added pads -->
+		<!-- added pads
 		<visual>
 			<origin xyz="0 -0.04 0.38"/>
@@ -459,6 +488,7 @@
 			</geometry>
 		</collision>
-		<xacro:inertial_box mass="${leg_mass}" x="0.04" y="0.04" z="0.4">
-			<origin xyz="0 0 0" rpy="0 0 0"/>
+		-->
+		<xacro:inertial_box mass="${leg_mass3}" x="0.04" y="0.04" z="0.4">
+			<origin xyz="0 -0.04 0.18" rpy="0 0 0"/>
 		</xacro:inertial_box>
 	</link>
@@ -468,4 +498,8 @@
 		<mu2 value="${mu2}"/>
 		<fdir1 value="${fdir}"/>
+		<maxVel>1.0</maxVel>
+    	<minDepth>0.01</minDepth>
+		<kp>1000000.0</kp>
+ 		<kd>100.0</kd>
 	</gazebo>
 	<ros2_control name="GazeboSystem" type="system">
