Commit message: added control for custom model

File: description/robot.urdf.xacro (robot description, xacro)
@@ -1,5 +1,6 @@
 <?xml version="1.0"?>
 <robot xmlns:xacro="http://www.ros.org/wiki/xacro"  name="robot">
-	<xacro:include filename="robot_core_lr.xacro"/>
+	<!--<xacro:include filename="robot_core_lr.xacro"/>-->
+	<xacro:include filename="robot_core_hr.xacro"/>
     <xacro:include filename="gazebo_control.xacro"/>
 </robot>

File: description/robot_core_hr.xacro (robot description, xacro)
@@ -1,7 +1,8 @@
 <?xml version="1.0"?>
-<!-- This URDF was automatically created by SolidWorks to URDF Exporter! Originally created by Stephen Brawner (brawner@gmail.com)
-     Commit Version: 1.6.0-1-g15f4949  Build Version: 1.6.7594.29634
-     For more information, please see http://wiki.ros.org/sw_urdf_exporter -->
 <robot xmlns:xacro="http://www.ros.org/wiki/xacro">
+  <xacro:property name="damping" value="1.0"/>
+  <xacro:property name="friction" value="1000.0"/>
+  <xacro:property name="mu1" value="100.0"/>
+  <xacro:property name="mu2" value="100.0"/>
   <link
     name="base_link">
@@ -44,4 +45,5 @@
     </collision>
   </link>
+  <!--FR1_LINK -->
   <link
     name="fr1_link">
@@ -95,11 +97,15 @@
       link="fr1_link" />
     <axis
-      xyz="0 0 -1" />
+      xyz="0 0 1" />
     <limit
       lower="${-pi/2}"
       upper="${pi/2}"
-      effort="0"
-      velocity="0" />
-  </joint>
+      effort="1.4"
+      velocity="1" />
+    <dynamics
+      damping="${damping}"
+      friction="${friction}" />
+  </joint>
+  <!--FR2_LINK -->
   <link
     name="fr2_link">
@@ -153,11 +159,15 @@
       link="fr2_link" />
     <axis
-      xyz="-0.0011869 0 1" />
+      xyz="-0.0011869 0 -1" />
     <limit
       lower="${-pi/2}"
       upper="${pi/2}"
-      effort="0"
-      velocity="0" />
-  </joint>
+      effort="1.4"
+      velocity="1" />
+    <dynamics
+      damping="${damping}"
+      friction="${friction}" />
+  </joint>
+  <!-- FR3_LINK -->
   <link
     name="fr3_link">
@@ -211,11 +221,15 @@
       link="fr3_link" />
     <axis
-      xyz="-0.0011869 0 1" />
+      xyz="-0.0011869 0 -1" />
     <limit
       lower="${-pi}"
       upper="${pi}"
-      effort="0"
-      velocity="0" />
-  </joint>
+      effort="1.4"
+      velocity="1" />
+    <dynamics
+      damping="${damping}"
+      friction="${friction}" />
+  </joint>
+  <!-- FL1_LINK -->
   <link
     name="fl1_link">
@@ -273,7 +287,11 @@
       lower="${-pi/2}"
       upper="${pi/2}"
-      effort="0"
-      velocity="0" />
-  </joint>
+      effort="1.4"
+      velocity="1" />
+    <dynamics
+      damping="${damping}"
+      friction="${friction}" />
+  </joint>
+  <!-- FL2_LINK -->
   <link
     name="fl2_link">
@@ -331,7 +349,11 @@
       lower="${-pi/2}"
       upper="${pi/2}"
-      effort="0"
-      velocity="0" />
-  </joint>
+      effort="1.4"
+      velocity="1" />
+    <dynamics
+      damping="${damping}"
+      friction="${friction}" />
+  </joint>
+  <!-- FL3_LINK -->
   <link
     name="fl3_link">
@@ -389,7 +411,11 @@
       lower="${-pi}"
       upper="${pi}"
-      effort="0"
-      velocity="0" />
-  </joint>
+      effort="1.4"
+      velocity="1" />
+    <dynamics
+      damping="${damping}"
+      friction="${friction}" />
+  </joint>
+  <!-- RR1_LINK -->
   <link
     name="rr1_link">
@@ -447,7 +473,11 @@
       lower="${-pi/2}"
       upper="${pi/2}"
-      effort="0"
-      velocity="0" />
-  </joint>
+      effort="1.4"
+      velocity="1" />
+    <dynamics
+      damping="${damping}"
+      friction="${friction}" />
+  </joint>
+  <!-- RR2_LINK -->
   <link
     name="rr2_link">
@@ -505,7 +535,11 @@
       lower="${-pi/2}"
       upper="${pi/2}"
-      effort="0"
-      velocity="0" />
-  </joint>
+      effort="1.4"
+      velocity="1" />
+    <dynamics
+      damping="${damping}"
+      friction="${friction}" />
+  </joint>
+  <!-- RR3_LINK -->
   <link
     name="rr3_link">
@@ -563,7 +597,11 @@
       lower="${-pi}"
       upper="${pi}"
-      effort="0"
-      velocity="0" />
-  </joint>
+      effort="1.4"
+      velocity="1" />
+    <dynamics
+      damping="${damping}"
+      friction="${friction}" />
+  </joint>
+  <!--RL1_LINK -->
   <link
     name="rl1_link">
@@ -617,11 +655,15 @@
       link="rl1_link" />
     <axis
-      xyz="0 0 -1" />
+      xyz="0 0 1" />
     <limit
       lower="${-pi/2}"
       upper="${pi/2}"
-      effort="0"
-      velocity="0" />
-  </joint>
+      effort="1.4"
+      velocity="1" />
+    <dynamics
+      damping="${damping}"
+      friction="${friction}" />
+  </joint>
+  <!-- RL2_LINK -->
   <link
     name="rl2_link">
@@ -675,11 +717,15 @@
       link="rl2_link" />
     <axis
-      xyz="0.010572 0 0.99994" />
+      xyz="0.010572 0 -0.99994" />
     <limit
       lower="${-pi/2}"
       upper="${pi/2}"
-      effort="0"
-      velocity="0" />
-  </joint>
+      effort="1.4"
+      velocity="1" />
+    <dynamics
+      damping="${damping}"
+      friction="${friction}" />
+  </joint>
+  <!-- RL3_LINK -->
   <link
     name="rl3_link">
@@ -733,10 +779,224 @@
       link="rl3_link" />
     <axis
-      xyz="0.010572 0 0.99994" />
+      xyz="0.010572 0 -0.99994" />
     <limit
       lower="${-pi}"
       upper="${pi}"
-      effort="0"
-      velocity="0" />
-  </joint>
+      effort="1.4"
+      velocity="1" />
+    <dynamics
+      damping="${damping}"
+      friction="${friction}" />
+  </joint>
+  <!-- GAZEBO REF -->
+  <gazebo reference="base_link">
+    <material>Gazebo/Red</material>
+    <minDepth>0.0002</minDepth>
+  </gazebo>
+  <gazebo reference="fr1_link">
+    <material>Gazebo/Black</material>
+    <maxVel>1.0</maxVel>
+  </gazebo>
+  <gazebo reference="fr2_link">
+    <material>Gazebo/Red</material>
+    <maxVel>1.0</maxVel>
+  </gazebo>
+  <gazebo reference="fr3_link">
+    <material>Gazebo/Black</material>
+    <mu1 value="${mu1}"/>
+    <mu2 value="${mu2}"/>
+    <maxVel>1.0</maxVel>
+    <minDepth>0.0002</minDepth>
+    <kp>1000000.0</kp>
+    <kd>100.0</kd>
+  </gazebo>
+  <gazebo reference="fl1_link">
+    <material>Gazebo/Black</material>
+    <maxVel>1.0</maxVel>
+  </gazebo>
+  <gazebo reference="fl2_link">
+    <material>Gazebo/Red</material>
+    <maxVel>1.0</maxVel>
+  </gazebo>
+  <gazebo reference="fl3_link">
+    <material>Gazebo/Black</material>
+    <mu1 value="${mu1}"/>
+    <mu2 value="${mu2}"/>
+    <maxVel>1.0</maxVel>
+    <minDepth>0.0002</minDepth>
+    <kp>1000000.0</kp>
+    <kd>100.0</kd>
+  </gazebo>
+  <gazebo reference="rr1_link">
+    <material>Gazebo/Black</material>
+    <maxVel>1.0</maxVel>
+  </gazebo>
+  <gazebo reference="rr2_link">
+    <material>Gazebo/Red</material>
+    <maxVel>1.0</maxVel>
+  </gazebo>
+  <gazebo reference="rr3_link">
+    <material>Gazebo/Black</material>
+    <mu1 value="${mu1}"/>
+    <mu2 value="${mu2}"/>
+    <maxVel>1.0</maxVel>
+    <minDepth>0.0002</minDepth>
+    <kp>1000000.0</kp>
+    <kd>100.0</kd>
+  </gazebo>
+  <gazebo reference="rl1_link">
+    <material>Gazebo/Black</material>
+    <maxVel>1.0</maxVel>
+  </gazebo>
+  <gazebo reference="rl2_link">
+    <material>Gazebo/Red</material>
+    <maxVel>1.0</maxVel>
+  </gazebo>
+  <gazebo reference="rl3_link">
+    <material>Gazebo/Black</material>
+    <mu1 value="${mu1}"/>
+    <mu2 value="${mu2}"/>
+    <maxVel>1.0</maxVel>
+    <minDepth>0.0002</minDepth>
+    <kp>1000000.0</kp>
+    <kd>100.0</kd>
+  </gazebo>
+  <!-- GAZEBO CONTROL -->
+  <ros2_control name="GazeboSystem" type="system">
+    <hardware>
+      <plugin>gazebo_ros2_control/GazeboSystem</plugin>
+    </hardware>
+    <joint name="fr1_joint">
+      <command_interface name="position">
+        <param name="min">${-pi/2}</param>
+        <param name="max">${pi/2}</param>
+      </command_interface>
+      <state_interface name="position">
+        <param name="initial_value">${0}</param>
+      </state_interface>
+      <state_interface name="velocity"/>
+      <state_interface name="effort"/>
+    </joint>
+    <joint name="fr2_joint">
+      <command_interface name="position">
+        <param name="min">${-pi/2}</param>
+        <param name="max">${pi/2}</param>
+      </command_interface>
+      <state_interface name="position">
+        <param name="initial_value">${0}</param>
+      </state_interface>
+      <state_interface name="velocity"/>
+      <state_interface name="effort"/>
+    </joint>
+    <joint name="fr3_joint">
+      <command_interface name="position">
+        <param name="min">${-pi}</param>
+        <param name="max">${pi}</param>
+      </command_interface>
+      <state_interface name="position">
+        <param name="initial_value">${0}</param>
+      </state_interface>
+      <state_interface name="velocity"/>
+      <state_interface name="effort"/>
+    </joint>
+    <joint name="fl1_joint">
+      <command_interface name="position">
+        <param name="min">${-pi/2}</param>
+        <param name="max">${pi/2}</param>
+      </command_interface>
+      <state_interface name="position">
+        <param name="initial_value">${0}</param>
+      </state_interface>
+      <state_interface name="velocity"/>
+      <state_interface name="effort"/>
+    </joint>
+    <joint name="fl2_joint">
+      <command_interface name="position">
+        <param name="min">${-pi/2}</param>
+        <param name="max">${pi/2}</param>
+      </command_interface>
+      <state_interface name="position">
+        <param name="initial_value">${0}</param>
+      </state_interface>
+      <state_interface name="velocity"/>
+      <state_interface name="effort"/>
+    </joint>
+    <joint name="fl3_joint">
+      <command_interface name="position">
+        <param name="min">${-pi}</param>
+        <param name="max">${pi}</param>
+      </command_interface>
+      <state_interface name="position">
+        <param name="initial_value">${0}</param>
+      </state_interface>
+      <state_interface name="velocity"/>
+      <state_interface name="effort"/>
+    </joint>
+    <joint name="rr1_joint">
+      <command_interface name="position">
+        <param name="min">${-pi/2}</param>
+        <param name="max">${pi/2}</param>
+      </command_interface>
+      <state_interface name="position">
+        <param name="initial_value">${0}</param>
+      </state_interface>
+      <state_interface name="velocity"/>
+      <state_interface name="effort"/>
+    </joint>
+    <joint name="rr2_joint">
+      <command_interface name="position">
+        <param name="min">${-pi/2}</param>
+        <param name="max">${pi/2}</param>
+      </command_interface>
+      <state_interface name="position">
+        <param name="initial_value">${0}</param>
+      </state_interface>
+      <state_interface name="velocity"/>
+      <state_interface name="effort"/>
+    </joint>
+    <joint name="rr3_joint">
+      <command_interface name="position">
+        <param name="min">${-pi}</param>
+        <param name="max">${pi}</param>
+      </command_interface>
+      <state_interface name="position">
+        <param name="initial_value">${0}</param>
+      </state_interface>
+      <state_interface name="velocity"/>
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
File: description/robot_core_lr.xacro (robot description, xacro)
@@ -3,13 +3,13 @@
 	<xacro:include filename="inertial_macros.xacro"/>
 	<xacro:property name="damping" value="10"/>
-	<xacro:property name="friction" value="500"/>
-	<xacro:property name="mu1" value="550"/>
-	<xacro:property name="mu2" value="550"/>
+	<xacro:property name="friction" value="100"/>
+	<xacro:property name="mu1" value="1"/>
+	<xacro:property name="mu2" value="1"/>
 	<xacro:property name="velocity" value="1"/>
 	<xacro:property name="effort" value="10"/>
-	<xacro:property name="base_mass" value="10"/>
-	<xacro:property name="leg_mass" value="5"/>
-	<xacro:property name="leg_mass3" value="5"/>
-	<xacro:property name="fdir" value="1 0 0"/>
+	<xacro:property name="base_mass" value="5"/>
+	<xacro:property name="leg_mass" value="1"/>
+	<xacro:property name="leg_mass3" value="1"/>
+	<xacro:property name="fdir" value="0 0 1"/>
 	<link name="base_link">
 	</link>
@@ -39,7 +39,4 @@
 	<gazebo reference="stand_link">
 		<material>Gazebo/Red</material>
-		<mu1 value="${mu1}"/>
-		<mu2 value="${mu2}"/>
-		<fdir1 value="${fdir}"/>
 		<maxVel>1.0</maxVel>
     	<minDepth>0.01</minDepth>
@@ -73,9 +70,5 @@
 	<gazebo reference="lleg1_ax1_link">
 		<material>Gazebo/Black</material>
-		<mu1 value="${mu1}"/>
-		<mu2 value="${mu2}"/>
-		<fdir1 value="${fdir}"/>
-		<maxVel>1.0</maxVel>
-    	<minDepth>0.01</minDepth>
+		<maxVel>1.0</maxVel>
 	</gazebo>
 	<!-- LEFT_LEG1_AX2 -->
@@ -107,9 +100,5 @@
 	<gazebo reference="lleg1_ax2_link">
 		<material>Gazebo/Red</material>
-		<mu1 value="${mu1}"/>
-		<mu2 value="${mu2}"/>
-		<fdir1 value="${fdir}"/>
-		<maxVel>1.0</maxVel>
-    	<minDepth>0.01</minDepth>
+		<maxVel>1.0</maxVel>
 	</gazebo>
 	<!-- LEFT_LEG1_AX3 -->
@@ -143,7 +132,7 @@
 		<mu1 value="${mu1}"/>
 		<mu2 value="${mu2}"/>
-		<fdir1 value="${fdir}"/>
-		<maxVel>1.0</maxVel>
-    	<minDepth>0.01</minDepth>
+		<!--<fdir1 value="${fdir}"/>-->
+		<maxVel>1.0</maxVel>
+    	<minDepth>0.04</minDepth>
 		<kp>1000000.0</kp>
 		<kd>100.0</kd>
@@ -177,9 +166,5 @@
 	<gazebo reference="lleg2_ax1_link">
 		<material>Gazebo/Black</material>
-		<mu1 value="${mu1}"/>
-		<mu2 value="${mu2}"/>
-		<fdir1 value="${fdir}"/>
-		<maxVel>1.0</maxVel>
-    	<minDepth>0.01</minDepth>
+		<maxVel>1.0</maxVel>
 	</gazebo>
 	<!-- LEFT_LEG2_AX2 -->
@@ -211,9 +196,5 @@
 	<gazebo reference="lleg2_ax2_link">
 		<material>Gazebo/Red</material>
-		<mu1 value="${mu1}"/>
-		<mu2 value="${mu2}"/>
-		<fdir1 value="${fdir}"/>
-		<maxVel>1.0</maxVel>
-    	<minDepth>0.01</minDepth>
+		<maxVel>1.0</maxVel>
 	</gazebo>
 	<!-- LEFT_LEG2_AX3 -->
@@ -239,18 +220,4 @@
 			</geometry>
 		</collision>
-		<!-- added pads
-		<visual>
-			<origin xyz="0 -0.04 0.38"/>
-			<geometry>
-				<sphere radius="0.04"/>
-			</geometry>
-		</visual>
-		<collision>
-			<origin xyz="0 -0.04 0.38"/>
-			<geometry>
-				<sphere radius="0.04"/>
-			</geometry>
-		</collision>
-		-->
 		<xacro:inertial_box mass="${leg_mass3}" x="0.04" y="0.04" z="0.4">
 			<origin xyz="0 -0.04 0.18" rpy="0 0 0"/>
@@ -261,7 +228,7 @@
 		<mu1 value="${mu1}"/>
 		<mu2 value="${mu2}"/>
-		<fdir1 value="${fdir}"/>
-		<maxVel>1.0</maxVel>
-    	<minDepth>0.01</minDepth>
+		<!--<fdir1 value="${fdir}"/>-->
+		<maxVel>1.0</maxVel>
+    	<minDepth>0.04</minDepth>
 		<kp>1000000.0</kp>
 		<kd>100.0</kd>
@@ -295,9 +262,5 @@
 	<gazebo reference="rleg1_ax1_link">
 		<material>Gazebo/Black</material>
-		<mu1 value="${mu1}"/>
-		<mu2 value="${mu2}"/>
-		<fdir1 value="${fdir}"/>
-		<maxVel>1.0</maxVel>
-    	<minDepth>0.01</minDepth>
+		<maxVel>1.0</maxVel>
 	</gazebo>
 	<!-- RIGHT_LEG1_AX2 -->
@@ -329,9 +292,5 @@
 	<gazebo reference="rleg1_ax2_link">
 		<material>Gazebo/Red</material>
-		<mu1 value="${mu1}"/>
-		<mu2 value="${mu2}"/>
-		<fdir1 value="${fdir}"/>
-		<maxVel>1.0</maxVel>
-    	<minDepth>0.01</minDepth>
+		<maxVel>1.0</maxVel>
 	</gazebo>
 	<!-- RIGHT_LEG1_AX3 -->
@@ -357,18 +316,4 @@
 			</geometry>
 		</collision>
-		<!-- added pads
-		<visual>
-			<origin xyz="0 -0.04 0.38"/>
-			<geometry>
-				<sphere radius="0.04"/>
-			</geometry>
-		</visual>
-		<collision>
-			<origin xyz="0 -0.04 0.38"/>
-			<geometry>
-				<sphere radius="0.04"/>
-			</geometry>
-		</collision>
-		-->
 		<xacro:inertial_box mass="${leg_mass3}" x="0.04" y="0.04" z="0.4">
 			<origin xyz="0 -0.04 0.18" rpy="0 0 0"/>
@@ -379,7 +324,7 @@
 		<mu1 value="${mu1}"/>
 		<mu2 value="${mu2}"/>
-		<fdir1 value="${fdir}"/>
-		<maxVel>1.0</maxVel>
-    	<minDepth>0.01</minDepth>
+		<!--<fdir1 value="${fdir}"/>-->
+		<maxVel>1.0</maxVel>
+    	<minDepth>0.04</minDepth>
 		<kp>1000000.0</kp>
 		<kd>100.0</kd>
@@ -413,9 +358,5 @@
 	<gazebo reference="rleg2_ax1_link">
 		<material>Gazebo/Black</material>
-		<mu1 value="${mu1}"/>
-		<mu2 value="${mu2}"/>
-		<fdir1 value="${fdir}"/>
-		<maxVel>1.0</maxVel>
-    	<minDepth>0.01</minDepth>
+		<maxVel>1.0</maxVel>
 	</gazebo>
 	<!-- RIGHT_LEG2_AX2 -->
@@ -447,9 +388,5 @@
 	<gazebo reference="rleg2_ax2_link">
 		<material>Gazebo/Red</material>
-		<mu1 value="${mu1}"/>
-		<mu2 value="${mu2}"/>
-		<fdir1 value="${fdir}"/>
-		<maxVel>1.0</maxVel>
-    	<minDepth>0.01</minDepth>
+		<maxVel>1.0</maxVel>
 	</gazebo>
 	<!-- RIGHT_LEG2_AX3 -->
@@ -475,18 +412,4 @@
 			</geometry>
 		</collision>
-		<!-- added pads
-		<visual>
-			<origin xyz="0 -0.04 0.38"/>
-			<geometry>
-				<sphere radius="0.04"/>
-			</geometry>
-		</visual>
-		<collision>
-			<origin xyz="0 -0.04 0.38"/>
-			<geometry>
-				<sphere radius="0.04"/>
-			</geometry>
-		</collision>
-		-->
 		<xacro:inertial_box mass="${leg_mass3}" x="0.04" y="0.04" z="0.4">
 			<origin xyz="0 -0.04 0.18" rpy="0 0 0"/>
@@ -497,7 +420,7 @@
 		<mu1 value="${mu1}"/>
 		<mu2 value="${mu2}"/>
-		<fdir1 value="${fdir}"/>
-		<maxVel>1.0</maxVel>
-    	<minDepth>0.01</minDepth>
+		<!--<fdir1 value="${fdir}"/>-->
+		<maxVel>1.0</maxVel>
+    	<minDepth>0.04</minDepth>
 		<kp>1000000.0</kp>
  		<kd>100.0</kd>
