Commit message: simple changes

File: description/robot_core_hr.xacro (robot description, xacro)
@@ -1,8 +1,10 @@
 <?xml version="1.0"?>
 <robot xmlns:xacro="http://www.ros.org/wiki/xacro">
-  <xacro:property name="damping" value="1.0"/>
-  <xacro:property name="friction" value="1000.0"/>
-  <xacro:property name="mu1" value="100.0"/>
-  <xacro:property name="mu2" value="100.0"/>
+  <xacro:property name="damping" value="0.7"/>
+  <xacro:property name="friction" value="100.0"/>
+  <xacro:property name="mu1" value="10000.0"/>
+  <xacro:property name="mu2" value="10000.0"/>
+  <xacro:property name="fdir" value="0 1 0"/>
+  <xacro:property name="minDepth" value="0.002"/>
   <link
     name="base_link">
@@ -792,13 +794,19 @@
   <gazebo reference="base_link">
     <material>Gazebo/Red</material>
-    <minDepth>0.0002</minDepth>
+    <minDepth>${minDepth}</minDepth>
+	<mu1 value="${mu1}"/>
+    <mu2 value="${mu2}"/>
   </gazebo>
   <gazebo reference="fr1_link">
     <material>Gazebo/Black</material>
     <maxVel>1.0</maxVel>
+	<mu1 value="${mu1}"/>
+    <mu2 value="${mu2}"/>
   </gazebo>
   <gazebo reference="fr2_link">
     <material>Gazebo/Red</material>
     <maxVel>1.0</maxVel>
+	<mu1 value="${mu1}"/>
+    <mu2 value="${mu2}"/>
   </gazebo>
   <gazebo reference="fr3_link">
@@ -806,6 +814,7 @@
     <mu1 value="${mu1}"/>
     <mu2 value="${mu2}"/>
+	<fdir1>${fdir}</fdir1>
     <maxVel>1.0</maxVel>
-    <minDepth>0.0002</minDepth>
+    <minDepth>${minDepth}</minDepth>
     <kp>1000000.0</kp>
     <kd>100.0</kd>
@@ -814,8 +823,12 @@
     <material>Gazebo/Black</material>
     <maxVel>1.0</maxVel>
+	<mu1 value="${mu1}"/>
+    <mu2 value="${mu2}"/>
   </gazebo>
   <gazebo reference="fl2_link">
     <material>Gazebo/Red</material>
     <maxVel>1.0</maxVel>
+	<mu1 value="${mu1}"/>
+    <mu2 value="${mu2}"/>
   </gazebo>
   <gazebo reference="fl3_link">
@@ -823,6 +836,7 @@
     <mu1 value="${mu1}"/>
     <mu2 value="${mu2}"/>
+	<fdir1>${fdir}</fdir1>
     <maxVel>1.0</maxVel>
-    <minDepth>0.0002</minDepth>
+    <minDepth>${minDepth}</minDepth>
     <kp>1000000.0</kp>
     <kd>100.0</kd>
@@ -831,8 +845,12 @@
     <material>Gazebo/Black</material>
     <maxVel>1.0</maxVel>
+	<mu1 value="${mu1}"/>
+    <mu2 value="${mu2}"/>
   </gazebo>
   <gazebo reference="rr2_link">
     <material>Gazebo/Red</material>
     <maxVel>1.0</maxVel>
+	<mu1 value="${mu1}"/>
+    <mu2 value="${mu2}"/>
   </gazebo>
   <gazebo reference="rr3_link">
@@ -840,6 +858,7 @@
     <mu1 value="${mu1}"/>
     <mu2 value="${mu2}"/>
+	<fdir1>${fdir}</fdir1>
     <maxVel>1.0</maxVel>
-    <minDepth>0.0002</minDepth>
+    <minDepth>${minDepth}</minDepth>
     <kp>1000000.0</kp>
     <kd>100.0</kd>
@@ -848,8 +867,12 @@
     <material>Gazebo/Black</material>
     <maxVel>1.0</maxVel>
+	<mu1 value="${mu1}"/>
+    <mu2 value="${mu2}"/>
   </gazebo>
   <gazebo reference="rl2_link">
     <material>Gazebo/Red</material>
     <maxVel>1.0</maxVel>
+	<mu1 value="${mu1}"/>
+    <mu2 value="${mu2}"/>
   </gazebo>
   <gazebo reference="rl3_link">
@@ -857,6 +880,7 @@
     <mu1 value="${mu1}"/>
     <mu2 value="${mu2}"/>
+	<fdir1>${fdir}</fdir1>
     <maxVel>1.0</maxVel>
-    <minDepth>0.0002</minDepth>
+    <minDepth>${minDepth}</minDepth>
     <kp>1000000.0</kp>
     <kd>100.0</kd>
@@ -872,4 +896,15 @@
         <param name="max">${pi/2}</param>
       </command_interface>
+      <command_interface name="velocity">
+        <param name="min">-1</param>
+        <param name="max">1</param>
+      </command_interface>
+      <command_interface name="effort">
+       	<param name="min">-0.5</param>
+        <param name="max">0.5</param>
+      </command_interface>
+	  <command_interface name="Kp"/>
+      <command_interface name="Kd"/>
+      <command_interface name="effort_limit"/>
       <state_interface name="position">
         <param name="initial_value">${0}</param>
@@ -883,4 +918,15 @@
         <param name="max">${pi/2}</param>
       </command_interface>
+      <command_interface name="velocity">
+        <param name="min">-1</param>
+        <param name="max">1</param>
+      </command_interface>
+      <command_interface name="effort">
+       	<param name="min">-0.5</param>
+        <param name="max">0.5</param>
+      </command_interface>
+	  <command_interface name="Kp"/>
+      <command_interface name="Kd"/>
+      <command_interface name="effort_limit"/>
       <state_interface name="position">
         <param name="initial_value">${0}</param>
@@ -894,4 +940,15 @@
         <param name="max">${pi}</param>
       </command_interface>
+      <command_interface name="velocity">
+        <param name="min">-1</param>
+        <param name="max">1</param>
+      </command_interface>
+      <command_interface name="effort">
+       	<param name="min">-0.5</param>
+        <param name="max">0.5</param>
+      </command_interface>
+	  <command_interface name="Kp"/>
+      <command_interface name="Kd"/>
+      <command_interface name="effort_limit"/>
       <state_interface name="position">
         <param name="initial_value">${0}</param>
@@ -905,4 +962,15 @@
         <param name="max">${pi/2}</param>
       </command_interface>
+      <command_interface name="velocity">
+        <param name="min">-1</param>
+        <param name="max">1</param>
+      </command_interface>
+      <command_interface name="effort">
+       	<param name="min">-0.5</param>
+        <param name="max">0.5</param>
+      </command_interface>
+	  <command_interface name="Kp"/>
+      <command_interface name="Kd"/>
+      <command_interface name="effort_limit"/>
       <state_interface name="position">
         <param name="initial_value">${0}</param>
@@ -916,4 +984,15 @@
         <param name="max">${pi/2}</param>
       </command_interface>
+      <command_interface name="velocity">
+        <param name="min">-1</param>
+        <param name="max">1</param>
+      </command_interface>
+      <command_interface name="effort">
+       	<param name="min">-0.5</param>
+        <param name="max">0.5</param>
+      </command_interface>
+	  <command_interface name="Kp"/>
+      <command_interface name="Kd"/>
+      <command_interface name="effort_limit"/>
       <state_interface name="position">
         <param name="initial_value">${0}</param>
@@ -927,4 +1006,15 @@
         <param name="max">${pi}</param>
       </command_interface>
+      <command_interface name="velocity">
+        <param name="min">-1</param>
+        <param name="max">1</param>
+      </command_interface>
+      <command_interface name="effort">
+       	<param name="min">-0.5</param>
+        <param name="max">0.5</param>
+      </command_interface>
+	  <command_interface name="Kp"/>
+      <command_interface name="Kd"/>
+      <command_interface name="effort_limit"/>
       <state_interface name="position">
         <param name="initial_value">${0}</param>
@@ -938,4 +1028,15 @@
         <param name="max">${pi/2}</param>
       </command_interface>
+      <command_interface name="velocity">
+        <param name="min">-1</param>
+        <param name="max">1</param>
+      </command_interface>
+      <command_interface name="effort">
+       	<param name="min">-0.5</param>
+        <param name="max">0.5</param>
+      </command_interface>
+	  <command_interface name="Kp"/>
+      <command_interface name="Kd"/>
+      <command_interface name="effort_limit"/>
       <state_interface name="position">
         <param name="initial_value">${0}</param>
@@ -949,4 +1050,15 @@
         <param name="max">${pi/2}</param>
       </command_interface>
+      <command_interface name="velocity">
+        <param name="min">-1</param>
+        <param name="max">1</param>
+      </command_interface>
+      <command_interface name="effort">
+       	<param name="min">-0.5</param>
+        <param name="max">0.5</param>
+      </command_interface>
+	  <command_interface name="Kp"/>
+      <command_interface name="Kd"/>
+      <command_interface name="effort_limit"/>
       <state_interface name="position">
         <param name="initial_value">${0}</param>
@@ -960,4 +1072,15 @@
         <param name="max">${pi}</param>
       </command_interface>
+      <command_interface name="velocity">
+        <param name="min">-1</param>
+        <param name="max">1</param>
+      </command_interface>
+      <command_interface name="effort">
+       	<param name="min">-0.5</param>
+        <param name="max">0.5</param>
+      </command_interface>
+	  <command_interface name="Kp"/>
+      <command_interface name="Kd"/>
+      <command_interface name="effort_limit"/>
       <state_interface name="position">
         <param name="initial_value">${0}</param>
@@ -971,4 +1094,15 @@
         <param name="max">${pi/2}</param>
       </command_interface>
+      <command_interface name="velocity">
+        <param name="min">-1</param>
+        <param name="max">1</param>
+      </command_interface>
+      <command_interface name="effort">
+       	<param name="min">-0.5</param>
+        <param name="max">0.5</param>
+      </command_interface>
+	  <command_interface name="Kp"/>
+      <command_interface name="Kd"/>
+      <command_interface name="effort_limit"/>
       <state_interface name="position">
         <param name="initial_value">${0}</param>
@@ -982,4 +1116,15 @@
         <param name="max">${pi/2}</param>
       </command_interface>
+      <command_interface name="velocity">
+        <param name="min">-1</param>
+        <param name="max">1</param>
+      </command_interface>
+      <command_interface name="effort">
+       	<param name="min">-0.5</param>
+        <param name="max">0.5</param>
+      </command_interface>
+	  <command_interface name="Kp"/>
+      <command_interface name="Kd"/>
+      <command_interface name="effort_limit"/>
       <state_interface name="position">
         <param name="initial_value">${0}</param>
@@ -993,4 +1138,15 @@
         <param name="max">${pi}</param>
       </command_interface>
+      <command_interface name="velocity">
+        <param name="min">-1</param>
+        <param name="max">1</param>
+      </command_interface>
+      <command_interface name="effort">
+       	<param name="min">-0.5</param>
+        <param name="max">0.5</param>
+      </command_interface>
+	  <command_interface name="Kp"/>
+      <command_interface name="Kd"/>
+      <command_interface name="effort_limit"/>
       <state_interface name="position">
         <param name="initial_value">${0}</param>
@@ -1000,3 +1156,123 @@
     </joint>
   </ros2_control>
+  <transmission name="tran1">
+    <type>transmission_interface/SimpleTransmission</type>
+    <joint name="fr1_joint">
+      <hardwareInterface>hardware_interface/EffortJointInterface</hardwareInterface>
+    </joint>
+    <actuator name="motor1">
+      <hardwareInterface>hardware_interface/EffortJointInterface</hardwareInterface>
+      <mechanicalReduction>5</mechanicalReduction>
+    </actuator>
+  </transmission>
+  <transmission name="tran2">
+    <type>transmission_interface/SimpleTransmission</type>
+    <joint name="fr2_joint">
+      <hardwareInterface>hardware_interface/EffortJointInterface</hardwareInterface>
+    </joint>
+    <actuator name="motor2">
+      <hardwareInterface>hardware_interface/EffortJointInterface</hardwareInterface>
+      <mechanicalReduction>5</mechanicalReduction>
+    </actuator>
+  </transmission>
+  <transmission name="tran3">
+    <type>transmission_interface/SimpleTransmission</type>
+    <joint name="fr3_joint">
+      <hardwareInterface>hardware_interface/EffortJointInterface</hardwareInterface>
+    </joint>
+    <actuator name="motor3">
+      <hardwareInterface>hardware_interface/EffortJointInterface</hardwareInterface>
+      <mechanicalReduction>5</mechanicalReduction>
+    </actuator>
+  </transmission>
+  <transmission name="tran4">
+    <type>transmission_interface/SimpleTransmission</type>
+    <joint name="fl1_joint">
+      <hardwareInterface>hardware_interface/EffortJointInterface</hardwareInterface>
+    </joint>
+    <actuator name="motor4">
+      <hardwareInterface>hardware_interface/EffortJointInterface</hardwareInterface>
+      <mechanicalReduction>5</mechanicalReduction>
+    </actuator>
+  </transmission>
+  <transmission name="tran5">
+    <type>transmission_interface/SimpleTransmission</type>
+    <joint name="fl2_joint">
+      <hardwareInterface>hardware_interface/EffortJointInterface</hardwareInterface>
+    </joint>
+    <actuator name="motor5">
+      <hardwareInterface>hardware_interface/EffortJointInterface</hardwareInterface>
+      <mechanicalReduction>5</mechanicalReduction>
+    </actuator>
+  </transmission>
+  <transmission name="tran6">
+    <type>transmission_interface/SimpleTransmission</type>
+    <joint name="fl3_joint">
+      <hardwareInterface>hardware_interface/EffortJointInterface</hardwareInterface>
+    </joint>
+    <actuator name="motor6">
+      <hardwareInterface>hardware_interface/EffortJointInterface</hardwareInterface>
+      <mechanicalReduction>5</mechanicalReduction>
+    </actuator>
+  </transmission>
+  <transmission name="tran7">
+    <type>transmission_interface/SimpleTransmission</type>
+    <joint name="rr1_joint">
+      <hardwareInterface>hardware_interface/EffortJointInterface</hardwareInterface>
+    </joint>
+    <actuator name="motor7">
+      <hardwareInterface>hardware_interface/EffortJointInterface</hardwareInterface>
+      <mechanicalReduction>5</mechanicalReduction>
+    </actuator>
+  </transmission>
+  <transmission name="tran8">
+    <type>transmission_interface/SimpleTransmission</type>
+    <joint name="rr2_joint">
+      <hardwareInterface>hardware_interface/EffortJointInterface</hardwareInterface>
+    </joint>
+    <actuator name="motor8">
+      <hardwareInterface>hardware_interface/EffortJointInterface</hardwareInterface>
+      <mechanicalReduction>5</mechanicalReduction>
+    </actuator>
+  </transmission>
+  <transmission name="tran9">
+    <type>transmission_interface/SimpleTransmission</type>
+    <joint name="rr3_joint">
+      <hardwareInterface>hardware_interface/EffortJointInterface</hardwareInterface>
+    </joint>
+    <actuator name="motor9">
+      <hardwareInterface>hardware_interface/EffortJointInterface</hardwareInterface>
+      <mechanicalReduction>5</mechanicalReduction>
+    </actuator>
+  </transmission>
+  <transmission name="tran10">
+    <type>transmission_interface/SimpleTransmission</type>
+    <joint name="rl1_joint">
+      <hardwareInterface>hardware_interface/EffortJointInterface</hardwareInterface>
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