Commit message: simple changes

File: description/robot_core_lr.xacro (robot description, xacro)
@@ -2,10 +2,10 @@
 <robot xmlns:xacro="http://www.ros.org/wiki/xacro">
 	<xacro:include filename="inertial_macros.xacro"/>
-	<xacro:property name="damping" value="10"/>
-	<xacro:property name="friction" value="100"/>
-	<xacro:property name="mu1" value="1"/>
-	<xacro:property name="mu2" value="1"/>
+	<xacro:property name="damping" value="0.7"/>
+	<xacro:property name="friction" value="10"/>
+	<xacro:property name="mu1" value="100"/>
+	<xacro:property name="mu2" value="100"/>
 	<xacro:property name="velocity" value="1"/>
-	<xacro:property name="effort" value="10"/>
+	<xacro:property name="effort" value="1.7"/>
 	<xacro:property name="base_mass" value="5"/>
 	<xacro:property name="leg_mass" value="1"/>
@@ -435,9 +435,21 @@
                 <param name="max">${pi/2}</param>
             </command_interface>
-            <state_interface name="position">
-                <param name="initial_value">${0}</param>
-            </state_interface>
-            <state_interface name="velocity"/>
-            <state_interface name="effort"/>
+			<command_interface name="velocity">
+        		<param name="min">-1</param>
+        		<param name="max">1</param>
+      		</command_interface>
+      		<command_interface name="effort">
+        		<param name="min">-0.5</param>
+        		<param name="max">0.5</param>
+      		</command_interface>
+			<command_interface name="Kp"/>
+      		<command_interface name="Kd"/>
+      		<command_interface name="effort_limit"/>
+            <state_interface name="position">
+                <param name="initial_value">${0}</param>
+            </state_interface>
+            <state_interface name="velocity"/>
+            <state_interface name="effort"/>
+			<state_interface name="contact_information"/>
         </joint>
 		<joint name="lleg1_ax2_joint">
@@ -446,9 +458,21 @@
                 <param name="max">${pi/2}</param>
             </command_interface>
-            <state_interface name="position">
-                <param name="initial_value">${0}</param>
-            </state_interface>
-            <state_interface name="velocity"/>
-            <state_interface name="effort"/>
+			<command_interface name="velocity">
+        		<param name="min">-1</param>
+        		<param name="max">1</param>
+      		</command_interface>
+      		<command_interface name="effort">
+        		<param name="min">-0.5</param>
+        		<param name="max">0.5</param>
+      		</command_interface>
+			<command_interface name="Kp"/>
+      		<command_interface name="Kd"/>
+      		<command_interface name="effort_limit"/>
+            <state_interface name="position">
+                <param name="initial_value">${0}</param>
+            </state_interface>
+            <state_interface name="velocity"/>
+            <state_interface name="effort"/>
+			<state_interface name="contact_information"/>
         </joint>
 		<joint name="lleg1_ax3_joint">
@@ -457,9 +481,21 @@
                 <param name="max">${pi}</param>
             </command_interface>
-            <state_interface name="position">
-                <param name="initial_value">${0}</param>
-            </state_interface>
-            <state_interface name="velocity"/>
-            <state_interface name="effort"/>
+			<command_interface name="velocity">
+        		<param name="min">-1</param>
+        		<param name="max">1</param>
+      		</command_interface>
+      		<command_interface name="effort">
+        		<param name="min">-0.5</param>
+        		<param name="max">0.5</param>
+      		</command_interface>
+			<command_interface name="Kp"/>
+      		<command_interface name="Kd"/>
+      		<command_interface name="effort_limit"/>
+            <state_interface name="position">
+                <param name="initial_value">${0}</param>
+            </state_interface>
+            <state_interface name="velocity"/>
+            <state_interface name="effort"/>
+			<state_interface name="contact_information"/>
         </joint>
 		<joint name="lleg2_ax1_joint">
@@ -468,9 +504,21 @@
                 <param name="max">${pi/2}</param>
             </command_interface>
-            <state_interface name="position">
-                <param name="initial_value">${0}</param>
-            </state_interface>
-            <state_interface name="velocity"/>
-            <state_interface name="effort"/>
+			<command_interface name="velocity">
+        		<param name="min">-1</param>
+        		<param name="max">1</param>
+      		</command_interface>
+      		<command_interface name="effort">
+        		<param name="min">-0.5</param>
+        		<param name="max">0.5</param>
+      		</command_interface>
+			<command_interface name="Kp"/>
+      		<command_interface name="Kd"/>
+      		<command_interface name="effort_limit"/>
+            <state_interface name="position">
+                <param name="initial_value">${0}</param>
+            </state_interface>
+            <state_interface name="velocity"/>
+            <state_interface name="effort"/>
+			<state_interface name="contact_information"/>
         </joint>
 		<joint name="lleg2_ax2_joint">
@@ -479,9 +527,21 @@
                 <param name="max">${pi/2}</param>
             </command_interface>
-            <state_interface name="position">
-                <param name="initial_value">${0}</param>
-            </state_interface>
-            <state_interface name="velocity"/>
-            <state_interface name="effort"/>
+			<command_interface name="velocity">
+        		<param name="min">-1</param>
+        		<param name="max">1</param>
+      		</command_interface>
+      		<command_interface name="effort">
+        		<param name="min">-0.5</param>
+        		<param name="max">0.5</param>
+      		</command_interface>
+			<command_interface name="Kp"/>
+      		<command_interface name="Kd"/>
+      		<command_interface name="effort_limit"/>
+            <state_interface name="position">
+                <param name="initial_value">${0}</param>
+            </state_interface>
+            <state_interface name="velocity"/>
+            <state_interface name="effort"/>
+			<state_interface name="contact_information"/>
         </joint>
 		<joint name="lleg2_ax3_joint">
@@ -490,9 +550,21 @@
                 <param name="max">${pi}</param>
             </command_interface>
-            <state_interface name="position">
-                <param name="initial_value">${0}</param>
-            </state_interface>
-            <state_interface name="velocity"/>
-            <state_interface name="effort"/>
+			<command_interface name="velocity">
+        		<param name="min">-1</param>
+        		<param name="max">1</param>
+      		</command_interface>
+      		<command_interface name="effort">
+        		<param name="min">-0.5</param>
+        		<param name="max">0.5</param>
+      		</command_interface>
+			<command_interface name="Kp"/>
+      		<command_interface name="Kd"/>
+      		<command_interface name="effort_limit"/>
+            <state_interface name="position">
+                <param name="initial_value">${0}</param>
+            </state_interface>
+            <state_interface name="velocity"/>
+            <state_interface name="effort"/>
+			<state_interface name="contact_information"/>
         </joint>
 		<joint name="rleg1_ax1_joint">
@@ -501,9 +573,21 @@
                 <param name="max">${pi/2}</param>
             </command_interface>
-            <state_interface name="position">
-                <param name="initial_value">${0}</param>
-            </state_interface>
-            <state_interface name="velocity"/>
-            <state_interface name="effort"/>
+			<command_interface name="velocity">
+        		<param name="min">-1</param>
+        		<param name="max">1</param>
+      		</command_interface>
+      		<command_interface name="effort">
+        		<param name="min">-0.5</param>
+        		<param name="max">0.5</param>
+      		</command_interface>
+			<command_interface name="Kp"/>
+     		<command_interface name="Kd"/>
+      		<command_interface name="effort_limit"/>
+            <state_interface name="position">
+                <param name="initial_value">${0}</param>
+            </state_interface>
+            <state_interface name="velocity"/>
+            <state_interface name="effort"/>
+			<state_interface name="contact_information"/>
         </joint>
 		<joint name="rleg1_ax2_joint">
@@ -512,9 +596,21 @@
                 <param name="max">${pi/2}</param>
             </command_interface>
-            <state_interface name="position">
-                <param name="initial_value">${0}</param>
-            </state_interface>
-            <state_interface name="velocity"/>
-            <state_interface name="effort"/>
+			<command_interface name="velocity">
+        		<param name="min">-1</param>
+        		<param name="max">1</param>
+      		</command_interface>
+      		<command_interface name="effort">
+        		<param name="min">-0.5</param>
+        		<param name="max">0.5</param>
+      		</command_interface>
+			<command_interface name="Kp"/>
+      		<command_interface name="Kd"/>
+      		<command_interface name="effort_limit"/>
+            <state_interface name="position">
+                <param name="initial_value">${0}</param>
+            </state_interface>
+            <state_interface name="velocity"/>
+            <state_interface name="effort"/>
+			<state_interface name="contact_information"/>
         </joint>
 		<joint name="rleg1_ax3_joint">
@@ -523,9 +619,21 @@
                 <param name="max">${pi}</param>
             </command_interface>
-            <state_interface name="position">
-                <param name="initial_value">${0}</param>
-            </state_interface>
-            <state_interface name="velocity"/>
-            <state_interface name="effort"/>
+			<command_interface name="velocity">
+        		<param name="min">-1</param>
+        		<param name="max">1</param>
+      		</command_interface>
+      		<command_interface name="effort">
+        		<param name="min">-0.5</param>
+        		<param name="max">0.5</param>
+      		</command_interface>
+			<command_interface name="Kp"/>
+      		<command_interface name="Kd"/>
+      		<command_interface name="effort_limit"/>
+            <state_interface name="position">
+                <param name="initial_value">${0}</param>
+            </state_interface>
+            <state_interface name="velocity"/>
+            <state_interface name="effort"/>
+			<state_interface name="contact_information"/>
         </joint>
 		<joint name="rleg2_ax1_joint">
@@ -534,9 +642,21 @@
                 <param name="max">${pi/2}</param>
             </command_interface>
-            <state_interface name="position">
-                <param name="initial_value">${0}</param>
-            </state_interface>
-            <state_interface name="velocity"/>
-            <state_interface name="effort"/>
+			<command_interface name="velocity">
+        		<param name="min">-1</param>
+        		<param name="max">1</param>
+      		</command_interface>
+      		<command_interface name="effort">
+        		<param name="min">-0.5</param>
+        		<param name="max">0.5</param>
+      		</command_interface>
+			<command_interface name="Kp"/>
+      		<command_interface name="Kd"/>
+      		<command_interface name="effort_limit"/>
+            <state_interface name="position">
+                <param name="initial_value">${0}</param>
+            </state_interface>
+            <state_interface name="velocity"/>
+            <state_interface name="effort"/>
+			<state_interface name="contact_information"/>
         </joint>
 		<joint name="rleg2_ax2_joint">
@@ -545,9 +665,21 @@
                 <param name="max">${pi/2}</param>
             </command_interface>
-            <state_interface name="position">
-                <param name="initial_value">${0}</param>
-            </state_interface>
-            <state_interface name="velocity"/>
-            <state_interface name="effort"/>
+			<command_interface name="velocity">
+        		<param name="min">-1</param>
+        		<param name="max">1</param>
+      		</command_interface>
+      		<command_interface name="effort">
+        		<param name="min">-0.5</param>
+        		<param name="max">0.5</param>
+      		</command_interface>
+			<command_interface name="Kp"/>
+      		<command_interface name="Kd"/>
+      		<command_interface name="effort_limit"/>
+            <state_interface name="position">
+                <param name="initial_value">${0}</param>
+            </state_interface>
+            <state_interface name="velocity"/>
+            <state_interface name="effort"/>
+			<state_interface name="contact_information"/>
         </joint>
 		<joint name="rleg2_ax3_joint">
@@ -556,9 +688,21 @@
                 <param name="max">${pi}</param>
             </command_interface>
-            <state_interface name="position">
-                <param name="initial_value">${0}</param>
-            </state_interface>
-            <state_interface name="velocity"/>
-            <state_interface name="effort"/>
+			<command_interface name="velocity">
+        		<param name="min">-1</param>
+        		<param name="max">1</param>
+      		</command_interface>
+      		<command_interface name="effort">
+        		<param name="min">-0.5</param>
+        		<param name="max">0.5</param>
+      		</command_interface>
+			<command_interface name="Kp"/>
+      		<command_interface name="Kd"/>
+      		<command_interface name="effort_limit"/>
+            <state_interface name="position">
+                <param name="initial_value">${0}</param>
+            </state_interface>
+            <state_interface name="velocity"/>
+            <state_interface name="effort"/>
+			<state_interface name="contact_information"/>
         </joint>
 	</ros2_control>

Commit message: update controller gain

File: description/robot_core_hr.xacro (robot description, xacro)
@@ -5,6 +5,8 @@
   <xacro:property name="mu1" value="10000.0"/>
   <xacro:property name="mu2" value="10000.0"/>
-  <xacro:property name="fdir" value="0 1 0"/>
+  <xacro:property name="fdir" value="0 0 1"/>
   <xacro:property name="minDepth" value="0.002"/>
+  <xacro:property name="kp" value="1000000"/>
+  <xacro:property name="kd" value="100"/>
   <link
     name="base_link">
@@ -817,6 +819,6 @@
     <maxVel>1.0</maxVel>
     <minDepth>${minDepth}</minDepth>
-    <kp>1000000.0</kp>
-    <kd>100.0</kd>
+    <kp>${kp}</kp>
+    <kd>${kd}</kd>
   </gazebo>
   <gazebo reference="fl1_link">
@@ -839,6 +841,6 @@
     <maxVel>1.0</maxVel>
     <minDepth>${minDepth}</minDepth>
-    <kp>1000000.0</kp>
-    <kd>100.0</kd>
+    <kp>${kp}</kp>
+    <kd>${kd}</kd>
   </gazebo>
   <gazebo reference="rr1_link">
@@ -861,6 +863,6 @@
     <maxVel>1.0</maxVel>
     <minDepth>${minDepth}</minDepth>
-    <kp>1000000.0</kp>
-    <kd>100.0</kd>
+    <kp>${kp}</kp>
+    <kd>${kd}</kd>
   </gazebo>
   <gazebo reference="rl1_link">
@@ -883,6 +885,6 @@
     <maxVel>1.0</maxVel>
     <minDepth>${minDepth}</minDepth>
-    <kp>1000000.0</kp>
-    <kd>100.0</kd>
+    <kp>${kp}</kp>
+    <kd>${kd}</kd>
   </gazebo>
   <!-- GAZEBO CONTROL -->
