Commit message: cleaning

File: description/robot_core_hr.xacro (robot description, xacro)
@@ -9,4 +9,5 @@
   <xacro:property name="kp" value="1000000"/>
   <xacro:property name="kd" value="100"/>
+  <xacro:property name="maxVel" value="3"/>
   <link
     name="base_link">
@@ -802,5 +803,5 @@
   <gazebo reference="fr1_link">
     <material>Gazebo/Black</material>
-    <maxVel>1.0</maxVel>
+    <maxVel>${maxVel}</maxVel>
 	<mu1 value="${mu1}"/>
     <mu2 value="${mu2}"/>
@@ -808,5 +809,5 @@
   <gazebo reference="fr2_link">
     <material>Gazebo/Red</material>
-    <maxVel>1.0</maxVel>
+    <maxVel>${maxVel}</maxVel>
 	<mu1 value="${mu1}"/>
     <mu2 value="${mu2}"/>
@@ -817,5 +818,5 @@
     <mu2 value="${mu2}"/>
 	<fdir1>${fdir}</fdir1>
-    <maxVel>1.0</maxVel>
+    <maxVel>${maxVel}</maxVel>
     <minDepth>${minDepth}</minDepth>
     <kp>${kp}</kp>
@@ -824,5 +825,5 @@
   <gazebo reference="fl1_link">
     <material>Gazebo/Black</material>
-    <maxVel>1.0</maxVel>
+    <maxVel>${maxVel}</maxVel>
 	<mu1 value="${mu1}"/>
     <mu2 value="${mu2}"/>
@@ -830,5 +831,5 @@
   <gazebo reference="fl2_link">
     <material>Gazebo/Red</material>
-    <maxVel>1.0</maxVel>
+    <maxVel>${maxVel}</maxVel>
 	<mu1 value="${mu1}"/>
     <mu2 value="${mu2}"/>
@@ -839,5 +840,5 @@
     <mu2 value="${mu2}"/>
 	<fdir1>${fdir}</fdir1>
-    <maxVel>1.0</maxVel>
+    <maxVel>${maxVel}</maxVel>
     <minDepth>${minDepth}</minDepth>
     <kp>${kp}</kp>
@@ -846,5 +847,5 @@
   <gazebo reference="rr1_link">
     <material>Gazebo/Black</material>
-    <maxVel>1.0</maxVel>
+    <maxVel>${maxVel}</maxVel>
 	<mu1 value="${mu1}"/>
     <mu2 value="${mu2}"/>
@@ -852,5 +853,5 @@
   <gazebo reference="rr2_link">
     <material>Gazebo/Red</material>
-    <maxVel>1.0</maxVel>
+    <maxVel>${maxVel}</maxVel>
 	<mu1 value="${mu1}"/>
     <mu2 value="${mu2}"/>
@@ -861,5 +862,5 @@
     <mu2 value="${mu2}"/>
 	<fdir1>${fdir}</fdir1>
-    <maxVel>1.0</maxVel>
+    <maxVel>${maxVel}</maxVel>
     <minDepth>${minDepth}</minDepth>
     <kp>${kp}</kp>
@@ -868,5 +869,5 @@
   <gazebo reference="rl1_link">
     <material>Gazebo/Black</material>
-    <maxVel>1.0</maxVel>
+    <maxVel>${maxVel}</maxVel>
 	<mu1 value="${mu1}"/>
     <mu2 value="${mu2}"/>
@@ -874,5 +875,5 @@
   <gazebo reference="rl2_link">
     <material>Gazebo/Red</material>
-    <maxVel>1.0</maxVel>
+    <maxVel>${maxVel}</maxVel>
 	<mu1 value="${mu1}"/>
     <mu2 value="${mu2}"/>
@@ -883,5 +884,5 @@
     <mu2 value="${mu2}"/>
 	<fdir1>${fdir}</fdir1>
-    <maxVel>1.0</maxVel>
+    <maxVel>${maxVel}</maxVel>
     <minDepth>${minDepth}</minDepth>
     <kp>${kp}</kp>
@@ -898,15 +899,4 @@
         <param name="max">${pi/2}</param>
       </command_interface>
-      <command_interface name="velocity">
-        <param name="min">-1</param>
-        <param name="max">1</param>
-      </command_interface>
-      <command_interface name="effort">
-       	<param name="min">-0.5</param>
-        <param name="max">0.5</param>
-      </command_interface>
-	  <command_interface name="Kp"/>
-      <command_interface name="Kd"/>
-      <command_interface name="effort_limit"/>
       <state_interface name="position">
         <param name="initial_value">${0}</param>
@@ -920,15 +910,4 @@
         <param name="max">${pi/2}</param>
       </command_interface>
-      <command_interface name="velocity">
-        <param name="min">-1</param>
-        <param name="max">1</param>
-      </command_interface>
-      <command_interface name="effort">
-       	<param name="min">-0.5</param>
-        <param name="max">0.5</param>
-      </command_interface>
-	  <command_interface name="Kp"/>
-      <command_interface name="Kd"/>
-      <command_interface name="effort_limit"/>
       <state_interface name="position">
         <param name="initial_value">${0}</param>
@@ -942,15 +921,4 @@
         <param name="max">${pi}</param>
       </command_interface>
-      <command_interface name="velocity">
-        <param name="min">-1</param>
-        <param name="max">1</param>
-      </command_interface>
-      <command_interface name="effort">
-       	<param name="min">-0.5</param>
-        <param name="max">0.5</param>
-      </command_interface>
-	  <command_interface name="Kp"/>
-      <command_interface name="Kd"/>
-      <command_interface name="effort_limit"/>
       <state_interface name="position">
         <param name="initial_value">${0}</param>
@@ -964,15 +932,4 @@
         <param name="max">${pi/2}</param>
       </command_interface>
-      <command_interface name="velocity">
-        <param name="min">-1</param>
-        <param name="max">1</param>
-      </command_interface>
-      <command_interface name="effort">
-       	<param name="min">-0.5</param>
-        <param name="max">0.5</param>
-      </command_interface>
-	  <command_interface name="Kp"/>
-      <command_interface name="Kd"/>
-      <command_interface name="effort_limit"/>
       <state_interface name="position">
         <param name="initial_value">${0}</param>
@@ -986,15 +943,4 @@
         <param name="max">${pi/2}</param>
       </command_interface>
-      <command_interface name="velocity">
-        <param name="min">-1</param>
-        <param name="max">1</param>
-      </command_interface>
-      <command_interface name="effort">
-       	<param name="min">-0.5</param>
-        <param name="max">0.5</param>
-      </command_interface>
-	  <command_interface name="Kp"/>
-      <command_interface name="Kd"/>
-      <command_interface name="effort_limit"/>
       <state_interface name="position">
         <param name="initial_value">${0}</param>
@@ -1008,15 +954,4 @@
         <param name="max">${pi}</param>
       </command_interface>
-      <command_interface name="velocity">
-        <param name="min">-1</param>
-        <param name="max">1</param>
-      </command_interface>
-      <command_interface name="effort">
-       	<param name="min">-0.5</param>
-        <param name="max">0.5</param>
-      </command_interface>
-	  <command_interface name="Kp"/>
-      <command_interface name="Kd"/>
-      <command_interface name="effort_limit"/>
       <state_interface name="position">
         <param name="initial_value">${0}</param>
@@ -1030,15 +965,4 @@
         <param name="max">${pi/2}</param>
       </command_interface>
-      <command_interface name="velocity">
-        <param name="min">-1</param>
-        <param name="max">1</param>
-      </command_interface>
-      <command_interface name="effort">
-       	<param name="min">-0.5</param>
-        <param name="max">0.5</param>
-      </command_interface>
-	  <command_interface name="Kp"/>
-      <command_interface name="Kd"/>
-      <command_interface name="effort_limit"/>
       <state_interface name="position">
         <param name="initial_value">${0}</param>
@@ -1052,15 +976,4 @@
         <param name="max">${pi/2}</param>
       </command_interface>
-      <command_interface name="velocity">
-        <param name="min">-1</param>
-        <param name="max">1</param>
-      </command_interface>
-      <command_interface name="effort">
-       	<param name="min">-0.5</param>
-        <param name="max">0.5</param>
-      </command_interface>
-	  <command_interface name="Kp"/>
-      <command_interface name="Kd"/>
-      <command_interface name="effort_limit"/>
       <state_interface name="position">
         <param name="initial_value">${0}</param>
@@ -1074,15 +987,4 @@
         <param name="max">${pi}</param>
       </command_interface>
-      <command_interface name="velocity">
-        <param name="min">-1</param>
-        <param name="max">1</param>
-      </command_interface>
-      <command_interface name="effort">
-       	<param name="min">-0.5</param>
-        <param name="max">0.5</param>
-      </command_interface>
-	  <command_interface name="Kp"/>
-      <command_interface name="Kd"/>
-      <command_interface name="effort_limit"/>
       <state_interface name="position">
         <param name="initial_value">${0}</param>
@@ -1096,15 +998,4 @@
         <param name="max">${pi/2}</param>
       </command_interface>
-      <command_interface name="velocity">
-        <param name="min">-1</param>
-        <param name="max">1</param>
-      </command_interface>
-      <command_interface name="effort">
-       	<param name="min">-0.5</param>
-        <param name="max">0.5</param>
-      </command_interface>
-	  <command_interface name="Kp"/>
-      <command_interface name="Kd"/>
-      <command_interface name="effort_limit"/>
       <state_interface name="position">
         <param name="initial_value">${0}</param>
@@ -1118,15 +1009,4 @@
         <param name="max">${pi/2}</param>
       </command_interface>
-      <command_interface name="velocity">
-        <param name="min">-1</param>
-        <param name="max">1</param>
-      </command_interface>
-      <command_interface name="effort">
-       	<param name="min">-0.5</param>
-        <param name="max">0.5</param>
-      </command_interface>
-	  <command_interface name="Kp"/>
-      <command_interface name="Kd"/>
-      <command_interface name="effort_limit"/>
       <state_interface name="position">
         <param name="initial_value">${0}</param>
@@ -1140,15 +1020,4 @@
         <param name="max">${pi}</param>
       </command_interface>
-      <command_interface name="velocity">
-        <param name="min">-1</param>
-        <param name="max">1</param>
-      </command_interface>
-      <command_interface name="effort">
-       	<param name="min">-0.5</param>
-        <param name="max">0.5</param>
-      </command_interface>
-	  <command_interface name="Kp"/>
-      <command_interface name="Kd"/>
-      <command_interface name="effort_limit"/>
       <state_interface name="position">
         <param name="initial_value">${0}</param>
